File: Schematics/Leduino/leduino.brd (EAGLE design)
At the start: 88.3 x 53.3 mm, 40 parts, among them U1 MIC39100-5.0WS, U10 DMN6040SSD, U3 DMN6040SSD, U4 DMN6040SSD, U5 DMN6040SSD, U6 DMN6040SSD, U7 DMN6040SSD, U8 DMN6040SSD, U9 DMN6040SSD

Commit message: Finished v2 update, ready for lbr cleanup
Parts:
- added 3.3V, 5V, A3: (no value), Leduino:SJ_2S-NO
- added U$6: (no value), Pro_Micro:OSHW-LOGO-M
- NC1, NC2, NC3, NC4: value PROTOBOARD5X4 -> PROTOBOARD6X4; device Leduino:5X4_PROTO -> Leduino:PROTOBOARD_6X4
- U$3: device Pro_Micro:OSHW-LOGO-M -> Pro_Micro:FIDUCIAL-1X2
- moved U$3 19.0 mm to (61.0, 34.9)
- moved NC1 4.45 mm to (6.35, 34.3)
- moved NC2 4.45 mm to (6.35, 19.1)
- moved NC3 1.91 mm to (21.6, 34.3)
- moved NC4 1.91 mm to (21.6, 19.1)
- moved A0 1.42 mm to (56.8, 27.9)
- moved A1 1.42 mm to (56.8, 25.4)
- moved A2 1.42 mm to (56.8, 22.9)
- moved RN2 0.90 mm to (57.5, 30.5)
- moved RN1 0.63 mm to (53.0, 24.8)
Connections:
- new net N$14: A3.1, RN1.5, U2.4
- net 3.3V: now also 3.3V.1
- net GND: no longer RN1.8, U2.4
- net N$15: now also RN1.8; no longer RN1.7
- net N$16: now also RN1.7; no longer RN1.6
- net N$21: now also RN1.6; no longer RN1.5
- net VCC: now also 3.3V.2, 5V.1, 5V.2, A3.2
Routing:
- net GND: track 72.1 -> 54.0 mm, vias 26 -> 30
- net N$14: track 0.00 -> 17.2 mm
- net VCC: track 77.3 -> 85.6 mm, vias 4 -> 5
- net 3.3V: track 3.81 -> 5.90 mm
- net N$15: track 10.3 -> 12.2 mm
- net N$16: track 11.0 -> 11.6 mm
Other:
- board text added: "YUN"
